File: pi-dmx.sch (EAGLE design)
At the start: 32 parts, among them IC4 74HCT08D, Q1 MMBTA56-SOT23, Q2 BCW71SMD, X1 MSTBV2, X2 NC3FBH2, X3 NC3MBH

Commit message: Added reset button and fixed connector layout
Parts:
- removed U$11: 1778780, grant:1778780
- added S2: (no value), switch-omron:10-XX
- added U$2: 1778780, grant:1778780
Connections:
- new net N$11: S2.P, S2.P1, U$1.RESET
- net EMISO: now also U$2.2; no longer U$11.2
- net ESCLK: now also U$2.3; no longer U$11.3
- net GND: now also S2.S, S2.S1, U$2.4; no longer U$11.4
- net N$10: now also U$2.1; no longer U$11.1
Other:
- moved on the sheet: R24, R27, X1-1
Changed lines of the file:
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@@
 <part name="SUPPLY28" library="supply2" deviceset="GND1" device=""/>
 <part name="SUPPLY26" library="supply2" deviceset="GND1" device=""/>
-<part name="U$11" library="grant" deviceset="1778780" device=""/>
 <part name="C10" library="microbuilder" deviceset="CAP_CERAMIC" device="0805" value="0.1uF"/>
 <part name="GND51" library="SparkFun-Aesthetics" deviceset="GND" device=""/>
@@
 <part name="D1" library="diode" deviceset="PESD1CAN" device=""/>
 <part name="SUPPLY5" library="supply2" deviceset="GND1" device=""/>
+<part name="S2" library="switch-omron" deviceset="10-XX" device=""/>
+<part name="GND6" library="SparkFun-Aesthetics" deviceset="GND" device=""/>
+<part name="GND7" library="SparkFun-Aesthetics" deviceset="GND" device=""/>
+<part name="U$2" library="grant" deviceset="1778780" device=""/>
 </parts>
 <sheets>
@@
 <instance part="POWER2" gate="G$1" x="127" y="86.36"/>
 <instance part="GND5" gate="1" x="127" y="73.66"/>
+<instance part="S2" gate="1" x="15.24" y="127" rot="R90"/>
+<instance part="GND6" gate="1" x="10.16" y="124.46"/>
+<instance part="GND7" gate="1" x="10.16" y="127"/>
 </instances>
 <busses>
@@
 <wire x1="127" y1="76.2" x2="127" y2="81.28" width="0.1524" layer="91"/>
 </segment>
+<segment>
+<pinref part="S2" gate="1" pin="S"/>
+<pinref part="GND6" gate="1" pin="GND"/>
+</segment>
+<segment>
+<pinref part="S2" gate="1" pin="S1"/>
+<pinref part="GND7" gate="1" pin="GND"/>
+</segment>
 </net>
 <net name="N$30" class="0">
@@
 <wire x1="91.44" y1="114.3" x2="127" y2="114.3" width="0.1524" layer="91"/>
 <wire x1="127" y1="114.3" x2="127" y2="104.14" width="0.1524" layer="91"/>
+</segment>
+</net>
+<net name="N$11" class="0">
+<segment>
+<pinref part="U$1" gate="G$1" pin="RESET"/>
+<pinref part="S2" gate="1" pin="P1"/>
+<wire x1="27.94" y1="129.54" x2="20.32" y2="129.54" width="0.1524" layer="91"/>
+<pinref part="S2" gate="1" pin="P"/>
+<wire x1="20.32" y1="127" x2="20.32" y2="129.54" width="0.1524" layer="91"/>
+<junction x="20.32" y="129.54"/>
 </segment>
 </net>
@@
 </plain>
 <instances>
-<instance part="U$11" gate="G$1" x="210.82" y="53.34"/>
 <instance part="GND2" gate="1" x="205.74" y="58.42"/>
-<instance part="X1" gate="-1" x="165.1" y="58.42"/>
+<instance part="X1" gate="-1" x="182.88" y="58.42"/>
 <instance part="X1" gate="-2" x="182.88" y="68.58"/>
-<instance part="GND3" gate="1" x="177.8" y="55.88"/>
+<instance part="GND3" gate="1" x="195.58" y="55.88"/>
 <instance part="EXT-PWR" gate="A" x="193.04" y="86.36"/>
 <instance part="P+1" gate="VCC" x="195.58" y="78.74" rot="R180"/>
+<instance part="U$2" gate="G$1" x="210.82" y="58.42"/>
 </instances>
 <busses>
@@
 <net name="GND" class="0">
 <segment>
-<pinref part="U$11" gate="G$1" pin="4"/>
-<pinref part="GND2" gate="1" pin="GND"/>
-</segment>
-<segment>
 <pinref part="GND3" gate="1" pin="GND"/>
 <pinref part="X1" gate="-1" pin="1"/>
-<wire x1="170.18" y1="58.42" x2="177.8" y2="58.42" width="0.1524" layer="91"/>
+<wire x1="187.96" y1="58.42" x2="195.58" y2="58.42" width="0.1524" layer="91"/>
+</segment>
+<segment>
+<pinref part="GND2" gate="1" pin="GND"/>
+<pinref part="U$2" gate="G$1" pin="4"/>
 </segment>
 </net>
 <net name="EMISO" class="0">
 <segment>
-<pinref part="U$11" gate="G$1" pin="2"/>
 <wire x1="205.74" y1="66.04" x2="193.04" y2="66.04" width="0.1524" layer="91"/>
 <label x="193.04" y="66.04" size="1.778" layer="95"/>
+<pinref part="U$2" gate="G$1" pin="2"/>
 </segment>
 </net>
 <net name="ESCLK" class="0">
 <segment>
-<pinref part="U$11" gate="G$1" pin="3"/>
 <wire x1="205.74" y1="63.5" x2="193.04" y2="63.5" width="0.1524" layer="91"/>
 <label x="193.04" y="63.5" size="1.778" layer="95"/>
+<pinref part="U$2" gate="G$1" pin="3"/>
 </segment>
 </net>
 <net name="N$10" class="0">
 <segment>
-<pinref part="U$11" gate="G$1" pin="1"/>
 <pinref part="X1" gate="-2" pin="1"/>
 <wire x1="187.96" y1="68.58" x2="193.04" y2="68.58" width="0.1524" layer="91"/>
@@
 <junction x="193.04" y="68.58"/>
 <pinref part="EXT-PWR" gate="A" pin="1"/>
+<pinref part="U$2" gate="G$1" pin="1"/>
 </segment>
 </net>
@@
 <instance part="IC4" gate="A" x="15.24" y="73.66"/>
 <instance part="IC4" gate="B" x="15.24" y="58.42"/>
-<instance part="R24" gate="G$1" x="38.1" y="63.5"/>
-<instance part="R27" gate="G$1" x="38.1" y="58.42"/>
+<instance part="R24" gate="G$1" x="35.56" y="73.66"/>
+<instance part="R27" gate="G$1" x="35.56" y="58.42"/>
 </instances>
 <busses>
@@
 <wire x1="7.62" y1="71.12" x2="-10.16" y2="71.12" width="0.1524" layer="91"/>
 <junction x="7.62" y="71.12"/>
-<label x="-10.16" y="73.66" size="1.778" layer="95"/>
+<label x="-10.16" y="71.628" size="1.778" layer="95"/>
 </segment>
 </net>
 <net name="N$89" class="0">
 <segment>
-<wire x1="33.02" y1="63.5" x2="22.86" y2="73.66" width="0.1524" layer="91"/>
+<wire x1="30.48" y1="73.66" x2="22.86" y2="73.66" width="0.1524" layer="91"/>
 <pinref part="IC4" gate="A" pin="O"/>
 <pinref part="R24" gate="G$1" pin="1"/>
@@
 <pinref part="R27" gate="G$1" pin="1"/>
 <pinref part="IC4" gate="B" pin="O"/>
-<wire x1="22.86" y1="58.42" x2="33.02" y2="58.42" width="0.1524" layer="91"/>
+<wire x1="22.86" y1="58.42" x2="30.48" y2="58.42" width="0.1524" layer="91"/>
 </segment>
 </net>
@@
 <pinref part="IC4" gate="B" pin="I0"/>
 <wire x1="7.62" y1="55.88" x2="7.62" y2="60.96" width="0.1524" layer="91"/>
-<wire x1="7.62" y1="55.88" x2="-12.7" y2="55.88" width="0.1524" layer="91"/>
+<wire x1="7.62" y1="55.88" x2="-10.16" y2="55.88" width="0.1524" layer="91"/>
 <junction x="7.62" y="55.88"/>
-<label x="-12.7" y="55.88" size="1.778" layer="95"/>
+<label x="-10.16" y="55.88" size="1.778" layer="95"/>
 </segment>
 </net>
@@
 <segment>
 <pinref part="R24" gate="G$1" pin="2"/>
-<wire x1="43.18" y1="63.5" x2="53.34" y2="63.5" width="0.1524" layer="91"/>
+<wire x1="40.64" y1="73.66" x2="53.34" y2="73.66" width="0.1524" layer="91"/>
+<label x="45.72" y="73.66" size="1.778" layer="95"/>
 </segment>
 </net>
@@
 <segment>
 <pinref part="R27" gate="G$1" pin="2"/>
-<wire x1="43.18" y1="58.42" x2="53.34" y2="58.42" width="0.1524" layer="91"/>
-</segment>
-</net>
+<wire x1="40.64" y1="58.42" x2="53.34" y2="58.42" width="0.1524" layer="91"/>
+<label x="45.72" y="58.42" size="1.778" layer="95"/>
+</segment>
+</net>

Commit message: Raspberry Pi 3 version
Parts:
- removed EXT-PWR: (no value), jumper:JP1E
- removed POWER1, POWER2: (no value), SparkFun-LED:LED1206
- removed Q1: MMBTA56-SOT23, transistor-pnp:MMBTA56-SOT23
- removed Q2: BCW71SMD, transistor-npn:BCW71SMD
- removed R24, R27: 100R, SparkFun-Passives:RESISTOR0603-RES
- removed R3, R4: 10K, SparkFun-Passives:RESISTOR0603-RES
- removed R6: 330R, SparkFun-Passives:RESISTOR0603-RES
- removed S1: 219-02, switch-dil:219-02
- removed S2: (no value), switch-omron:10-XX
- removed U$1: RPI-B-V2SHIELD, raspberry:RPI-B-V2SHIELD
- removed U$2: 1778780, grant:1778780
- removed U$7: MAX485SO8, hartmodems:MAX485SO8
- added C1: 1uF, microbuilder:CAP_CERAMIC0805
- added C11, C4, C9: 0.1uF, SparkFun-Capacitors:CAP0603-CAP
- added C2: 0.1uF, SparkFun-Passives:CAP0603-CAP
- added C5, C6: 10N, SparkFun-Capacitors:CAP0603-CAP
- added D2, D8: 250mA/100V, SparkFun-DiscreteSemi:DIODEBAS16
- added D3, D4, D5, D7: MMBZ5221BS_MMBZ5259BS, m-pad-2.1:MMBZ5221BS_MMBZ5259BS
- added D6: PESD1CAN, diode:PESD1CAN
- added IC1: MAX488CSA, maxim:MAX488CSA
- added IC2: 74AC139D, 74xx-eu:74AC139D
- added IC3: 74HC540DW, 74xx-eu:74HC540DW
- added PCB1: RPI2, e14_Rpi2_RevA:RPI2
- added R12, R13: 1M, SparkFun-Resistors:RESISTOR0603-RES
- added R14, R15: 330R, SparkFun-Resistors:RESISTOR0603-RES
- added RN1, RN2: 100R, resistor-dil:4R-NEXBS8V
- added RX, TX: (no value), SparkFun-LED:LED1206
- added U2: SN74LVC2G157-DCT, m-pad-2.1:SN74LVC2G157-DCT
- added X4: STRIP1, con-phoenix-254:MPT3
- added X5: STRIP2, con-phoenix-254:MPT3
- added X6: STRIP3, con-phoenix-254:MPT3
- added X7: STRIP4, con-phoenix-254:MPT3
- C3: value 1uF -> 0.1uF; device microbuilder:CAP_CERAMIC0805 -> SparkFun-Capacitors:CAP0603-CAP
- IC4: value 74HCT08D -> 74HC14D; device logic:74HCT08D -> 74xx-eu:74HC14D
- R1: device SparkFun-Passives:RESISTOR0603-RES -> SparkFun-Resistors:RESISTOR1206
- R2: value 10K -> 120R; device SparkFun-Passives:RESISTOR0603-RES -> SparkFun-Resistors:RESISTOR1206
- R5: value 330R -> 10K
- X1: value MSTBV2 -> 5V; device con-phoenix-508:MSTBV2 -> con-phoenix-254:MPT2
Connections:
- removed net EMISO: R27.2, U$2.2
- removed net ESCLK: R24.2, U$2.3
- removed net N$89: IC4A.O, R24.1
- new net +3V3: C7.P$2, PCB1.3V3@1, U$8.EN1, U$8.VDD1
- new net CE0: IC2A.A, IC2B.A, PCB1.CE0
- new net CE1: IC2A.B, IC2B.B, PCB1.CE1
- new net MISO0: D7.2.C, RN1B.2, X4-3.1
- new net MISO1: D3.2.C, RN1D.2, X5-3.1
- new net MISO2: D5.2.C, RN2B.2, X6-3.1
- new net MISO3: D4.2.C, RN2D.2, X7-3.1
- new net N$12: IC3A.Y4, RN1D.1
- new net N$13: IC2A.Y0, IC3A.A1
- new net N$14: IC2A.Y1, IC3A.A3
- new net N$15: IC2A.Y2, IC3A.A5
- new net N$16: IC2A.Y3, IC3A.A7
- new net N$17: IC2B.Y0, IC3A.A2
- new net N$18: IC2B.Y1, IC3A.A4
- new net N$20: IC2B.Y3, IC3A.A8
- new net N$21: C6.1, D2.C, IC4D.I, R12.2
- new net N$27: IC4B.O, TX.C
- new net N$32: IC3A.Y5, RN2A.1
- new net N$33: IC3A.Y6, RN2B.1
- new net N$34: IC3A.Y7, RN2C.1
- new net N$35: IC3A.Y8, RN2D.1
- new net SCLK0: D7.1.C, RN1A.2, X4-2.1
- new net SCLK1: D3.1.C, RN1C.2, X5-2.1
- new net SCLK2: D5.1.C, RN2A.2, X6-2.1
- new net SCLK3: D4.1.C, RN2C.2, X7-2.1
- net 5V: now also C1.P$2, C11.1, C2.2, C9.1, IC1P.VCC, IC4P.VCC, R14.2, R15.2, R22.2, U2.VCC; no longer C3.P$2, Q1.E, S1.4, U$7.VCC
- net DIRECTION: now also PCB1.GPIO17, R5.2; no longer U$1.UART0_RTS/GPIO17
- net GND: now also C3.1, C4.1, D3.1.A, D3.2.A, D4.1.A, D4.2.A, D5.1.A, D5.2.A, D7.1.A, D7.2.A, IC2P.GND, IC3A.G1, IC3A.G2, IC3P.GND, PCB1.GND@14, PCB1.GND@25, PCB1.GND@30, PCB1.GND@39, PCB1.GND@6, PCB1.GND@9, R5.1, X4-1.1, X5-1.1, X6-1.1, X7-1.1; no longer POWER1.C, POWER2.C, S2.S, S2.S1, U$1.GND, U$2.4
- net GND1: now also C1.P$1, C11.2, C2.1, C5.2, C6.2, C9.2, D6.3, IC1P.GND, IC4P.GND, R12.1, R13.1, R23.1, U2.#G, U2.GND; no longer C3.P$1, Q2.E, U$7.GND
- net MISO: now also IC2B.G, PCB1.MISO; no longer IC4B.I0, IC4B.I1, U$1.GPIO9/SPI0_MISO
- net N$1: now also D2.A, IC4C.O; no longer R5.1, U$1.GPIO27
- net N$10: now also C5.1, D8.C, IC4B.I, R13.2; no longer EXT-PWR.1, U$2.1, X1-2.1
- net N$11: now also IC3A.Y3, RN1C.1; no longer S2.P, S2.P1, U$1.RESET
- net N$19: now also IC2B.Y2, IC3A.A6; no longer IC4B.O, R27.1
- net N$2: now also D8.A, IC4A.O; no longer POWER1.A, R5.2
- net N$22: now also IC1G$1.Y, R1.2; no longer S1.2, U$7.A, X3.3
- net N$23: now also IC1G$1.Z; no longer U$7.B, X3.2
- net N$24: now also R14.1, RX.A; no longer U$7.DI, U$8.B2
- net N$25: now also IC4D.O, RX.C; no longer Q1.C, R22.2
- net N$26: now also R15.1, TX.A; no longer Q2.C, R23.1
- net N$28: now also IC1G$1.RO, IC4C.I, U2.B; no longer U$7.RO
- net N$3: now also D6.1, IC1G$1.B, R2.1, X3.2; no longer R1.2, S1.3
- net N$4: now also U$8.B1, U2.#A/B; no longer R2.2, R3.2, R4.2, S1.1
- net N$5: now also U$8.B2, U2.A; no longer U$7.DE, U$7.RE, U$8.B1
- net N$6: now also D6.2, IC1G$1.A, R2.2, X3.3; no longer Q1.B, R3.1
- net N$7: now also IC3A.Y2, RN1B.1; no longer Q2.B, R4.1
- net N$8: now also IC1G$1.DI, IC4A.I, U2.Y; no longer POWER2.A, R6.2
- net N$9: now also IC3A.Y1, RN1A.1; no longer R6.1, U$1.GPIO22
- net RX: now also PCB1.RX; no longer U$1.UART0_RXD/GPIO15
- net SCLK: now also IC2A.G, PCB1.CLK; no longer IC4A.I0, IC4A.I1, U$1.GPIO11/SPI0_SLCK
- net TX: now also PCB1.TX; no longer U$1.UART0_TXD/GPIO14
- net VCC: now also C3.2, C4.2, IC2P.VCC, IC3P.VCC, PCB1.5V@2, PCB1.5V@4, X1-2.1; no longer C7.P$2, EXT-PWR.2, U$1.+5V, U$8.EN1, U$8.VDD1
